File: Hardware/WatchSchematic.brd (EAGLE design)
At the start: 46 x 35 mm, 105 parts, among them IC1 BQ25180YBGR_BQ25180YBGR, IC2 DRV2605YZFR_DRV2605YZFR, IC3 BMA423_BMA423, IC9 RT6160AWSC_RT6160AWSC, J1 503480-2400_503480-2400, J2 TC2030-IDC_TC2030-IDC, J4 KH-TYPE-C-16P_KH-TYPE-C-16P, Q1 20V/4.2A/52mΩ/1.4W, Q3 ESP32_C6_LIBRARY_6_SI1308EDL-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, U1 NORDIC_NRF_4_NRF52840_QF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

Commit message: all done
Parts:
- moved TP_SWO 35.1 mm to (48.3, 126.0)
- moved TP_SWDCLK 34.4 mm to (52.0, 125.1)
- moved TP_RESET 31.5 mm to (46.7, 123.6)
- moved TP_3.3V 30.8 mm to (43.7, 122.4)
- moved TP_SWDIO 29.6 mm to (52.1, 128.1)
- moved C2-EP-DR 23.2 mm to (28.5, 118.6), turned to 90 degrees
- moved EDP_C9 18.2 mm to (31.5, 147.7)
- moved Q3 14.7 mm to (32.1, 139.1)
- moved EDP_C5 14.0 mm to (35.5, 129.9), turned to 180 degrees
- moved EDP_C12 10.9 mm to (19.3, 141.7)
- moved C5 10.8 mm to (49.5, 118.8)
- moved R4 9.32 mm to (53.0, 148.0)
- moved L2 8.92 mm to (46.3, 135.3), turned to 180 degrees
- moved EDP_C11 8.74 mm to (15.4, 148.9)
- moved L1 8.65 mm to (55.2, 127.1)
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Routing:
- net GND: track 39.7 -> 1693.3 mm, vias 0 -> 43
- net 3V3/2.4A: track 15.0 -> 105.5 mm, vias 0 -> 7
- net P0.01/XL2: track 0.00 -> 53.7 mm, vias 0 -> 4
- net SWDCLK: track 0.00 -> 49.2 mm, vias 0 -> 4
- net PREVGL: track 0.00 -> 48.7 mm, vias 0 -> 2
- net SWDIO: track 0.00 -> 43.3 mm, vias 0 -> 2
- net RESET: track 0.00 -> 37.1 mm, vias 0 -> 4
- net DEC4_6: track 0.00 -> 36.2 mm, vias 0 -> 5
- net N$3: track 0.00 -> 33.6 mm, vias 0 -> 2
- net P1.02/1.6C: track 0.00 -> 32.6 mm, vias 0 -> 3
- net EPD_3V3: track 0.00 -> 31.9 mm, vias 0 -> 2
- net N$29: track 0.00 -> 29.8 mm
- net SCL/2.4C: track 2.26 -> 32.0 mm, vias 0 -> 4
- net N$9: track 0.00 -> 29.7 mm, vias 0 -> 4
- net VBUS/1.5D: track 0.00 -> 29.0 mm
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- added copper zone on layer 1, net GND
- added copper zone on layer 16, net GND
- removed copper zone on layer 2, net GND
Other:
- outline, holes or cut-outs redrawn
