File: Hardware/WatchSchematic.sch (EAGLE design)
At the start: 105 parts, among them IC1 BQ25180YBGR_BQ25180YBGR, IC2 DRV2605YZFR_DRV2605YZFR, IC3 BMA423_BMA423, IC9 RT6160AWSC_RT6160AWSC, J1 503480-2400_503480-2400, J2 TC2030-IDC_TC2030-IDC, J4 KH-TYPE-C-16P_KH-TYPE-C-16P, Q1 20V/4.2A/52mΩ/1.4W, Q3 ESP32_C6_LIBRARY_6_SI1308EDL-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, U1 NORDIC_NRF_4_NRF52840_QF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

Commit message: solved issues
Other:
- note added: "Buttons"
- note added: "DC/DC"
- note added: "E-Paper Display Connector"
- note added: "E-Paper Drive Circuit"
- note added: "Fuel Gauge"
- note added: "Haptic Driver"
- note added: "IMU"
- note added: "LiPo Charger"
- note added: "SWD"
- note added: "USB C Connector & ESD Protection"
Changed lines of the file:
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@@
 <sheet>
 <plain>
+<text x="137.16" y="0" size="5.08" layer="97">SWD</text>
+<text x="-157.48" y="-5.08" size="5.08" layer="97">IMU</text>
+<text x="-154.94" y="99.06" size="5.08" layer="97">DC/DC</text>
+<text x="-142.24" y="162.56" size="5.08" layer="97">LiPo Charger</text>
 </plain>
 <instances>
@@
 <sheet>
 <plain>
+<text x="-175.26" y="111.76" size="5.08" layer="97">E-Paper Drive Circuit</text>
+<text x="53.34" y="91.44" size="5.08" layer="97">Haptic
+Driver</text>
+<text x="68.58" y="45.72" size="5.08" layer="97">Buttons</text>
+<text x="-15.24" y="38.1" size="5.08" layer="97">Fuel Gauge</text>
+<text x="-157.48" y="-12.7" size="5.08" layer="97">E-Paper Display Connector</text>
+<text x="-43.18" y="-33.02" size="5.08" layer="97">USB C Connector &amp; ESD
+Protection</text>
 </plain>
 <instances>
@@
 </drawing>
 <compatibility>
+<note version="6.3" minversion="6.2.2" severity="warning">
+Since Version 6.2.2 text objects can contain more than one line,
+which will not be processed correctly with this version.
+</note>
 <note version="8.3" severity="warning">
 Since Version 8.3, EAGLE supports the association of 3D packages
